File: hw-adapter-card.kicad_sch (KiCad schematic)
At the start: 28 parts, among them J1 Conn_01x12_Pin, J2 Conn_01x12_Pin, J3 DB25_Pins, J4 Conn_01x12_Pin, J5 Conn_01x12_Pin, U1 SN74LVC16244ADGGR, U2 OPA350, U3 SN74LVC32A

Commit message: erc clrean
Parts:
- removed C2, C3, C4, C5, C6: 100n, symbol Capacitor_Protonica:C_voltage
- removed J1, J2, J4, J5: Conn_01x12_Pin, symbol Connector:Conn_01x12_Pin
- removed JP1, JP2: SolderJumper_2_Open, symbol Jumper:SolderJumper_2_Open
- removed TP1, TP2, TP3, TP4, TP5, TP6, TP7, TP8: TestPoint, symbol Connector:TestPoint
- removed U1: SN74LVC16244ADGGR, symbol Buffer_Protonica:SN74LVC16244ADGGR
- removed U2: OPA350, symbol Device:Opamp_Dual
- removed U3: SN74LVC32A, symbol Logic_Gates_Protonica:SN74LVC32A
- added D1: SMAJ12A, Diode_SMD:D_SMA, symbol Diode:SMAJ12A
- added D2: SMAJ5.0A, Diode_SMD:D_SMA, symbol Diode:SMAJ5.0A
- added R10, R11, R5, R6, R7, R8, R9: 22R, symbol Device:R
- added U1, U2, U3: USBLC6-4SC6, Package_TO_SOT_SMD:SOT-23-6, symbol Power_Protection:USBLC6-4SC6
- R1, R3: value 0R -> 22R
- R2, R4: value DNP -> 22R
- renumbered J3 to J1
Connections:
- net CTRL.VIDEO_X is gone; now on an unnamed net: R1.1
- net CTRL.VIDEO_Y is gone; now on an unnamed net: R3.1
- net +2V5: now also C1.1, J1.1, J1.14 (P14), U2.6 (I/O4)
- net +3V3: now also J1.18 (P18), J1.5, D2.1 (A1), U1.5 (VBUS), U2.5 (VBUS), U3.5 (VBUS); no longer C1.1
- net GND: now also J1.12, J1.15 (P15), J1.16 (P16), J1.17 (P17), J1.21 (P21), J1.22 (P22), J1.23 (P23), J1.7, D1.2 (A2), D2.2 (A2), U1.2 (GND), U2.2 (GND), U3.2 (GND); no longer R2.2, R4.2
- net at R4.1: now also J1.11, U1.1 (I/O1); no longer R3.2
- net at J1.10: now also R5.1, U3.6 (I/O4)
- net at J1.13: now also U1.6 (I/O4)
- net +12V: now reaches J1.19 (P19)
- net +12V: now also J1.6, D1.1 (A1)
- net at J1.2: now also R11.1, U2.1 (I/O1)
- net at J1.20 (P20): now also R8.1, U3.1 (I/O1)
- net at J1.24 (P24): now also U1.3 (I/O2)
- net at J1.25 (P25): now also R2.1, U1.4 (I/O3)
- net at J1.3: now also R10.1, U2.3 (I/O2)
- net at J1.4: now also R9.1, U2.4 (I/O3)
- net at J1.8: now also R7.1, U3.3 (I/O2)
- net at J1.9: now also R6.1, U3.4 (I/O3)
- net LED_SERIAL.DATA: now reaches R1.2
- net LED_SERIAL.DATA: no longer R2.1
- new net LED_SERIAL.LE: R3.2
- new net LED_SERIAL.SCK: R2.2
- new net LED_SERIAL.~{OE}: R4.2
- new net PD_CTRL.CLK: R6.2
- new net PD_CTRL.EOS: R8.2
- new net PD_CTRL.GAIN: R10.2
- new net PD_CTRL.RST: R5.2
- new net PD_CTRL.TRG: R9.2
- new net PD_CTRL.VIDEO_12: R11.2
- new net PD_CTRL.VIDEO_34: R7.2
- no-connect marks 4 -> 0
Other:
- added sheet LED Driver (led_driver.kicad_sch)
- added sheet Photodiode Array Interface (photodiode_interface.kicad_sch)
- note removed: "CLK"
- note removed: "EOS"
- note removed: "EXTSP"
- note removed: "GAIN"
- note removed: "GND"
- note removed: "RESET"
- note removed: "TRG"
- note removed: "VDD"
- note removed: "VIDEO"
- note removed: "VMS"
- note removed: "VPD"
- note removed: "VREF"
- moved on the sheet: J1
