File: hw-front-end.kicad_pcb (KiCad board)
At the start: 6 copper layers, 150 x 65 mm, 74 parts, among them J102 DSUB-25, J201 Conn_02x04_Pin, J202 Conn_02x04_Pin, J301 Conn_02x06_Pin, J302 Conn_02x06_Pin, J303 Conn_02x06_Pin, J304 Conn_02x06_Pin, U101 USBLC6-4SC6, U102 USBLC6-4SC6, U103 USBLC6-4SC6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

Commit message: updated bom, ready for ordering
Parts:
- U301: value OPA350 -> OPA2350
Changed lines of the file:
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@@
 			(plot_on_all_layers_selection 0x00000000_00000000_00000000_00000000)
 			(disableapertmacros no)
-			(usegerberextensions no)
+			(usegerberextensions yes)
 			(usegerberattributes yes)
 			(usegerberadvancedattributes yes)
-			(creategerberjobfile yes)
+			(creategerberjobfile no)
 			(dashed_line_dash_ratio 12)
 			(dashed_line_gap_ratio 3)
@@
 			(outputformat 1)
 			(mirror no)
-			(drillshape 1)
+			(drillshape 0)
 			(scaleselection 1)
-			(outputdirectory "")
+			(outputdirectory "Output/Gerbers/")
 		)
 	)
@@
 			)
 		)
-		(property "Description" "CONN HEADER VERTICAL 12POS 2.54MM"
+		(property "Description" "CONN HEADER VERT 12POS 2.54MM"
 			(at 0 0 90)
 			(layer "F.Fab")
@@
 			)
 		)
-		(property "MPN" "G800W590018EU"
+		(property "MPN" "M20-9760642"
 			(at 0 0 90)
 			(unlocked yes)
@@
 			)
 		)
-		(property "Manufacturer" "Amphenol ICC"
+		(property "Manufacturer" "Harwin Inc."
 			(at 0 0 90)
 			(unlocked yes)
@@
 			)
 		)
-		(property "Description" "CONN HEADER VERTICAL 12POS 2.54MM"
+		(property "Description" "CONN HEADER VERT 12POS 2.54MM"
 			(at 0 0 90)
 			(layer "F.Fab")
@@
 			)
 		)
-		(property "MPN" "G800W590018EU"
+		(property "MPN" "M20-9760642"
 			(at 0 0 90)
 			(unlocked yes)
@@
 			)
 		)
-		(property "Manufacturer" "Amphenol ICC"
+		(property "Manufacturer" "Harwin Inc."
 			(at 0 0 90)
 			(unlocked yes)
@@
 			)
 		)
-		(property "Value" "OPA350"
+		(property "Value" "OPA2350"
 			(at 0 3.4 0)
 			(layer "F.Fab")
@@
 			)
 		)
-		(property "Datasheet" ""
+		(property "Datasheet" "https://www.ti.com/lit/ds/symlink/opa350.pdf?HQS=dis-dk-null-digikeymode-dsf-pf-null-wwe&ts=1781176353355&ref_url=https%253A%252F%252Fwww.ti.com%252Fgeneral%252Fdocs%252Fsuppproductinfo.tsp%253FdistId%253D10%2526gotoUrl%253Dhttps%253A%252F%252Fwww.ti.com%252Flit%252Fgpn%252Fopa350"
 			(at 0 0 0)
 			(layer "F.Fab")
@@
 			)
 		)
-		(property "MPN" "OPA350UA/2K5"
+		(property "MPN" "OPA2350UA/2K5"
 			(at 0 0 0)
 			(unlocked yes)
@@
 			)
 		)
-		(property "KLC_S3.3" ""
-			(at 0 0 0)
-			(unlocked yes)
-			(layer "F.Fab")
-			(hide yes)
-			(effects
-				(font
-					(size 1 1)
-					(thickness 0.15)
-				)
-			)
-		)
-		(property "KLC_S5.1" ""
-			(at 0 0 0)
-			(unlocked yes)
-			(layer "F.Fab")
-			(hide yes)
-			(effects
-				(font
-					(size 1 1)
-					(thickness 0.15)
-				)
-			)
-		)
 		(property ki_fp_filters "SOIC*3.9x4.9mm*P1.27mm* DIP*W7.62mm* MSOP*3x3mm*P0.65mm* SSOP*2.95x2.8mm*P0.65mm* TSSOP*3x3mm*P0.65mm* VSSOP*P0.5mm* TO?99*")
 		(sheetname "/Photodiode Array Interface/")
@@
 			)
 		)
-		(property "Description" "CONN HEADER VERTICAL 12POS 2.54MM"
+		(property "Description" "CONN HEADER VERT 12POS 2.54MM"
 			(at 0 0 90)
 			(layer "F.Fab")
@@
 			)
 		)
-		(property "MPN" "G800W590018EU"
+		(property "MPN" "M20-9760642"
 			(at 0 0 90)
 			(unlocked yes)
@@
 			)
 		)
-		(property "Manufacturer" "Amphenol ICC"
+		(property "Manufacturer" "Harwin Inc."
 			(at 0 0 90)
 			(unlocked yes)
@@
 			)
 		)
-		(property "Description" "CONN HEADER VERTICAL 8POS 2.54MM"
+		(property "Description" "CONN HEADER VERT 8POS 2.54MM"
 			(at 0 0 0)
 			(layer "F.Fab")
@@
 			)
 		)
-		(property "MPN" "PR20204VBDN"
+		(property "MPN" "M20-9760442"
 			(at 0 0 0)
 			(unlocked yes)
@@
 			)
 		)
-		(property "Manufacturer" "METZ CONNECT"
+		(property "Manufacturer" "Harwin Inc."
 			(at 0 0 0)
 			(unlocked yes)
@@
 			)
 		)
-		(property "Description" "CONN HEADER VERTICAL 12POS 2.54MM"
+		(property "Description" "CONN HEADER VERT 12POS 2.54MM"
 			(at 0 0 90)
 			(layer "F.Fab")
@@
 			)
 		)
-		(property "MPN" "G800W590018EU"
+		(property "MPN" "M20-9760642"
 			(at 0 0 90)
 			(unlocked yes)
@@
 			)
 		)
-		(property "Manufacturer" "Amphenol ICC"
+		(property "Manufacturer" "Harwin Inc."
 			(at 0 0 90)
 			(unlocked yes)
@@
 			)
 		)
-		(property "Description" "CONN HEADER VERTICAL 8POS 2.54MM"
+		(property "Description" "CONN HEADER VERT 8POS 2.54MM"
 			(at 0 0 0)
 			(layer "F.Fab")
@@
 			)
 		)
-		(property "MPN" "PR20204VBDN"
+		(property "MPN" "M20-9760442"
 			(at 0 0 0)
 			(unlocked yes)
@@
 			)
 		)
-		(property "Manufacturer" "METZ CONNECT"
+		(property "Manufacturer" "Harwin Inc."
 			(at 0 0 0)
 			(unlocked yes)
