File: photodiode_interface.kicad_sch (KiCad schematic)
At the start: 38 parts, among them J301 Conn_02x06_Pin, J302 Conn_02x06_Pin, J303 Conn_02x06_Pin, J304 Conn_02x06_Pin, U301 OPA350, U302 SN74LVC16244ADGGR, U303 74LVC2G32

Commit message: updated bom, ready for ordering
Parts:
- J301, J302, J303, J304: MPN G800W590018EU -> M20-9760642; Manufacturer Amphenol ICC -> Harwin Inc.
- U301: value OPA350 -> OPA2350; MPN OPA350UA/2K5 -> OPA2350UA/2K5
Changed lines of the file:
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@@
 			)
 		)
-		(property "Description" "CONN HEADER VERTICAL 12POS 2.54MM"
+		(property "Description" "CONN HEADER VERT 12POS 2.54MM"
 			(at 379.73 57.15 0)
 			(hide yes)
@@
 			)
 		)
-		(property "MPN" "G800W590018EU"
+		(property "MPN" "M20-9760642"
 			(at 379.73 57.15 0)
 			(hide yes)
@@
 			)
 		)
-		(property "Manufacturer" "Amphenol ICC"
+		(property "Manufacturer" "Harwin Inc."
 			(at 379.73 57.15 0)
 			(hide yes)
@@
 			)
 		)
-		(property "Value" "OPA350"
+		(property "Value" "OPA2350"
 			(at 176.53 54.61 0)
 			(show_name no)
@@
 			)
 		)
-		(property "Datasheet" ""
+		(property "Datasheet" "https://www.ti.com/lit/ds/symlink/opa350.pdf?HQS=dis-dk-null-digikeymode-dsf-pf-null-wwe&ts=1781176353355&ref_url=https%253A%252F%252Fwww.ti.com%252Fgeneral%252Fdocs%252Fsuppproductinfo.tsp%253FdistId%253D10%2526gotoUrl%253Dhttps%253A%252F%252Fwww.ti.com%252Flit%252Fgpn%252Fopa350"
 			(at 176.53 62.23 0)
 			(hide yes)
@@
 			)
 		)
-		(property "MPN" "OPA350UA/2K5"
+		(property "MPN" "OPA2350UA/2K5"
 			(at 176.53 62.23 0)
 			(hide yes)
@@
 			)
 		)
-		(property "KLC_S3.3" ""
-			(at 176.53 62.23 0)
-			(hide yes)
-			(show_name no)
-			(do_not_autoplace no)
-			(effects
-				(font
-					(size 1.27 1.27)
-				)
-			)
-		)
-		(property "KLC_S5.1" ""
-			(at 176.53 62.23 0)
-			(hide yes)
-			(show_name no)
-			(do_not_autoplace no)
-			(effects
-				(font
-					(size 1.27 1.27)
-				)
-			)
-		)
 		(pin "6"
 		)
@@
 			)
 		)
-		(property "Description" "CONN HEADER VERTICAL 12POS 2.54MM"
+		(property "Description" "CONN HEADER VERT 12POS 2.54MM"
 			(at 379.73 102.87 0)
 			(hide yes)
@@
 			)
 		)
-		(property "MPN" "G800W590018EU"
+		(property "MPN" "M20-9760642"
 			(at 379.73 102.87 0)
 			(hide yes)
@@
 			)
 		)
-		(property "Manufacturer" "Amphenol ICC"
+		(property "Manufacturer" "Harwin Inc."
 			(at 379.73 102.87 0)
 			(hide yes)
@@
 			)
 		)
-		(property "Description" "CONN HEADER VERTICAL 12POS 2.54MM"
+		(property "Description" "CONN HEADER VERT 12POS 2.54MM"
 			(at 379.73 153.67 0)
 			(hide yes)
@@
 			)
 		)
-		(property "MPN" "G800W590018EU"
+		(property "MPN" "M20-9760642"
 			(at 379.73 153.67 0)
 			(hide yes)
@@
 			)
 		)
-		(property "Manufacturer" "Amphenol ICC"
+		(property "Manufacturer" "Harwin Inc."
 			(at 379.73 153.67 0)
 			(hide yes)
@@
 			)
 		)
-		(property "Description" "CONN HEADER VERTICAL 12POS 2.54MM"
+		(property "Description" "CONN HEADER VERT 12POS 2.54MM"
 			(at 379.73 199.39 0)
 			(hide yes)
@@
 			)
 		)
-		(property "MPN" "G800W590018EU"
+		(property "MPN" "M20-9760642"
 			(at 379.73 199.39 0)
 			(hide yes)
@@
 			)
 		)
-		(property "Manufacturer" "Amphenol ICC"
+		(property "Manufacturer" "Harwin Inc."
 			(at 379.73 199.39 0)
 			(hide yes)
@@
 			)
 		)
-		(property "Value" "OPA350"
+		(property "Value" "OPA2350"
 			(at 176.53 25.4 0)
 			(show_name no)
@@
 			)
 		)
-		(property "Datasheet" ""
+		(property "Datasheet" "https://www.ti.com/lit/ds/symlink/opa350.pdf?HQS=dis-dk-null-digikeymode-dsf-pf-null-wwe&ts=1781176353355&ref_url=https%253A%252F%252Fwww.ti.com%252Fgeneral%252Fdocs%252Fsuppproductinfo.tsp%253FdistId%253D10%2526gotoUrl%253Dhttps%253A%252F%252Fwww.ti.com%252Flit%252Fgpn%252Fopa350"
 			(at 176.53 33.02 0)
 			(hide yes)
@@
 			)
 		)
-		(property "MPN" "OPA350UA/2K5"
+		(property "MPN" "OPA2350UA/2K5"
 			(at 176.53 33.02 0)
 			(hide yes)
@@
 			)
 		)
-		(property "KLC_S3.3" ""
-			(at 176.53 33.02 0)
-			(hide yes)
-			(show_name no)
-			(do_not_autoplace no)
-			(effects
-				(font
-					(size 1.27 1.27)
-				)
-			)
-		)
-		(property "KLC_S5.1" ""
-			(at 176.53 33.02 0)
-			(hide yes)
-			(show_name no)
-			(do_not_autoplace no)
-			(effects
-				(font
-					(size 1.27 1.27)
-				)
-			)
-		)
 		(pin "6"
 		)
@@
 			)
 		)
-		(property "Value" "OPA350"
+		(property "Value" "OPA2350"
 			(at 119.38 48.2599 0)
 			(show_name no)
@@
 			)
 		)
-		(property "Datasheet" ""
+		(property "Datasheet" "https://www.ti.com/lit/ds/symlink/opa350.pdf?HQS=dis-dk-null-digikeymode-dsf-pf-null-wwe&ts=1781176353355&ref_url=https%253A%252F%252Fwww.ti.com%252Fgeneral%252Fdocs%252Fsuppproductinfo.tsp%253FdistId%253D10%2526gotoUrl%253Dhttps%253A%252F%252Fwww.ti.com%252Flit%252Fgpn%252Fopa350"
 			(at 118.11 46.99 0)
 			(hide yes)
@@
 			)
 		)
-		(property "MPN" "OPA350UA/2K5"
+		(property "MPN" "OPA2350UA/2K5"
 			(at 118.11 46.99 0)
 			(hide yes)
@@
 			(at 118.11 46.99 0)
 			(hide yes)
-			(show_name no)
-			(do_not_autoplace no)
-			(effects
-				(font
-					(size 1.27 1.27)
-				)
-			)
-		)
-		(property "KLC_S3.3" ""
-			(at 118.11 46.99 0)
-			(hide yes)
-			(show_name no)
-			(do_not_autoplace no)
-			(effects
-				(font
-					(size 1.27 1.27)
-				)
-			)
-		)
-		(property "KLC_S5.1" ""
-			(at 118.11 46.99 0)
-			(hide yes)
